File: Pi_Breakout_Board.kicad_pcb (KiCad board)
At the start: 2 copper layers, 56.5 x 65 mm, 75 parts, among them J1 Raspberry_Pi_2_3, J2 Conn_02x04_Odd_Even heater he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, J3 Conn_02x08_Odd_Even thermisto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, J4 Screw_Terminal_01x02, J5 Conn_01x08_Male, J6 Conn_01x08_Male, J7 Conn_01x02_Female, J8 Conn_01x03_Male, Q1 Q_NMOS_GDSD, Q2 Q_NMOS_GDSD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

Commit message: Add 3V VCC pin to UART header (oops, shoulda had that). Other misc routing changes
Parts:
- J8: value Conn_01x03_Male -> Conn_01x04_Male; footprint Connector_PinHeader_2.54mm:PinHeader_1x03_P2.54mm_Vertical -> Connector_PinSocket_2.54mm:PinSocket_1x04_P2.54mm_Vertical
- moved J8 3.68 mm to (59.8, 130.8)
Connections:
- J1 pad 11: Net-(J1-Pad11) -> (no net)
- J1 pad 13: Net-(J1-Pad13) -> (no net)
- J1 pad 15: Net-(J1-Pad15) -> (no net)
- J1 pad 19: Net-(J1-Pad19) -> (no net)
- J1 pad 22: Net-(J1-Pad22) -> (no net)
- J1 pad 29: Net-(J1-Pad29) -> (no net)
- J1 pad 31: Net-(J1-Pad31) -> (no net)
- J1 pad 33: Net-(J1-Pad33) -> (no net)
- J1 pad 35: Net-(J1-Pad35) -> (no net)
- J1 pad 36: Net-(J1-Pad36) -> (no net)
- J1 pad 37: Net-(J1-Pad37) -> (no net)
- J1 pad 38: Net-(J1-Pad38) -> (no net)
- J1 pad 40: Net-(J1-Pad40) -> (no net)
- J1 pad 7: Net-(J1-Pad7) -> (no net)
- U1 pad 10: Net-(U1-Pad10) -> (no net)
- U1 pad 11: Net-(U1-Pad11) -> (no net)
- U1 pad 12: Net-(U1-Pad12) -> (no net)
- U1 pad 13: Net-(U1-Pad13) -> (no net)
- U1 pad 15: Net-(U1-Pad15) -> (no net)
- U1 pad 16: Net-(U1-Pad16) -> (no net)
- U1 pad 17: Net-(U1-Pad17) -> (no net)
- U1 pad 18: Net-(U1-Pad18) -> (no net)
- U1 pad 19: Net-(U1-Pad19) -> (no net)
- U1 pad 20: Net-(U1-Pad20) -> (no net)
- U1 pad 21: Net-(U1-Pad21) -> (no net)
- U1 pad 22: Net-(U1-Pad22) -> (no net)
- U2 pad 6: Net-(U2-Pad6) -> (no net)
Routing:
- net +3V3: track 204.6 -> 212.4 mm, vias 4 -> 5
- net RXD: track 14.9 -> 11.2 mm
- net TXD: track 18.5 -> 14.8 mm
- net SDA0: track 55.5 -> 54.2 mm
- net LED_YELLOW: track 57.1 -> 56.2 mm
- net LED_RED: track 59.6 -> 58.8 mm
- net LED_GREEN: track 57.3 -> 56.5 mm
- net GND: vias 11 -> 14
Other:
- board text added: "V"
