File: Pi_Breakout_Board.sch (KiCad schematic (older format))
At the start: 75 parts, among them J1 Raspberry_Pi_2_3, J2 Conn_02x04_Odd_Even heater he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, J3 Conn_02x08_Odd_Even thermisto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, J4 Screw_Terminal_01x02, J5 Conn_01x08_Male, J6 Conn_01x08_Male, J7 Conn_01x02_Female, J8 Conn_01x04_Male, Q1 Q_NMOS_GDSD, Q2 Q_NMOS_GDSD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

Commit message: Final commit before transfer to GA
Other:
- note added: "GA / Team OTheRS\nJacob Killelea"
- note removed: "Property GA/Team OTheRS"
Changed lines of the file:
@@
 	5150 4500 5150 4600
 NoConn ~ 4650 3600
-Text Notes 7200 6900 0    157  ~ 0
-Property GA/Team OTheRS
-Text Notes 7400 7500 0    50   ~ 0
+Text Notes 7050 7100 0    157  ~ 31
+GA / Team OTheRS\nJacob Killelea
+Text Notes 7350 7550 0    118  ~ 0
 Pi Breakout Board
 Text Notes 10600 7650 0    50   ~ 0
